File: schematics/m5-pantilt/m5-pantilt.sch (KiCad schematic (older format))
At the start: 11 parts, among them J1 Conn_02x15_Odd_Even, J2 Conn_02x03_Odd_Even, J3 Conn_02x03_Odd_Even, J4 Conn_01x04, J5 BAT, J6 Conn_01x04, SW1 SW_SPDT, U1 NL27WZ125

Commit message: Add jumper
Parts:
- added JP1, JP2: Jumper_3_Bridged12, Jumper:SolderJumper-3_P1.3mm_Bridged12_RoundedPad1.0x1.5mm, symbol Jumper:Jumper_3_Bridged12
- added R3, R4: 1k, Resistor_SMD:R_0603_1608Metric_Pad1.05x0.95mm_HandSolder, symbol Device:R
Connections:
- net PWM1: now reaches J1.19 (Pin_19)
- net PWM1: now also R3.2
- net PWM2: now reaches J1.20 (Pin_20)
- net PWM2: now also R4.2
- new net: J3.2 (Pin_2), J3.5 (Pin_5), JP1.1 (A), JP2.2 (C)
- new net: JP2.1 (A), R2.1
- new net: J2.2 (Pin_2), J2.5 (Pin_5), JP1.2 (C)
- new net: JP1.3 (B), R3.1
- new net: JP2.3 (B), R4.1
- no-connect marks 25 -> 23
Other:
- moved on the sheet: J2, J3
Changed lines of the file:
@@
 L Connector_Generic:Conn_02x03_Odd_Even J3
 U 1 1 60BD706E
-P 8550 4300
-F 0 "J3" H 8600 4617 50  0000 C CNN
-F 1 "Conn_02x03_Odd_Even" H 8600 4526 50  0000 C CNN
-F 2 "Connector_PinHeader_2.54mm:PinHeader_2x03_P2.54mm_Vertical" H 8550 4300 50  0001 C CNN
-F 3 "~" H 8550 4300 50  0001 C CNN
-	1    8550 4300
+P 9800 4300
+F 0 "J3" H 9850 4617 50  0000 C CNN
+F 1 "Conn_02x03_Odd_Even" H 9850 4526 50  0000 C CNN
+F 2 "Connector_PinHeader_2.54mm:PinHeader_2x03_P2.54mm_Vertical" H 9800 4300 50  0001 C CNN
+F 3 "~" H 9800 4300 50  0001 C CNN
+	1    9800 4300
 	1    0    0    -1
 $EndComp
@@
 Wire Wire Line
 	3450 4550 3550 4550
-Text Label 4800 5300 2    50   ~ 0
+Text Label 4950 5300 2    50   ~ 0
 RXD2
 Wire Wire Line
-	4800 5300 5400 5300
-Text Label 4800 5100 2    50   ~ 0
+	4950 5300 5400 5300
+Text Label 4950 5100 2    50   ~ 0
 TXD2
 Wire Wire Line
-	4800 5100 5400 5100
+	4950 5100 5400 5100
 $Comp
 L power:GND #PWR05
@@
 $EndComp
 Wire Wire Line
-	7200 5150 8000 5150
-Wire Wire Line
-	8000 4400 8350 4400
-Wire Wire Line
-	8000 4400 8000 4600
-Wire Wire Line
-	8000 4600 9100 4600
-Wire Wire Line
-	9100 4600 9100 4200
-Wire Wire Line
-	9100 4200 8850 4200
-Connection ~ 8000 4600
-Wire Wire Line
-	7300 4300 8350 4300
+	9250 4400 9400 4400
+Wire Wire Line
+	10350 4600 10350 4200
+Wire Wire Line
+	10350 4200 10100 4200
 Wire Wire Line
 	7300 2850 7300 3300
-NoConn ~ 8850 4300
-NoConn ~ 8850 4400
-Wire Wire Line
-	7550 4200 8350 4200
+NoConn ~ 10100 4300
+NoConn ~ 10100 4400
 $Comp
 L Connector_Generic:Conn_02x03_Odd_Even J2
 U 1 1 60C1A998
-P 8550 3600
-F 0 "J2" H 8600 3917 50  0000 C CNN
-F 1 "Conn_02x03_Odd_Even" H 8600 3826 50  0000 C CNN
-F 2 "Connector_PinHeader_2.54mm:PinHeader_2x03_P2.54mm_Vertical" H 8550 3600 50  0001 C CNN
-F 3 "~" H 8550 3600 50  0001 C CNN
-	1    8550 3600
-	1    0    0    -1
-$EndComp
-Wire Wire Line
-	8000 3700 8350 3700
-Wire Wire Line
-	8000 3900 9100 3900
-Wire Wire Line
-	7300 3600 8350 3600
-Wire Wire Line
-	7550 3500 8350 3500
-Wire Wire Line
-	8850 3500 9100 3500
-Wire Wire Line
-	9100 3500 9100 3900
-NoConn ~ 8850 3600
-NoConn ~ 8850 3700
-Wire Wire Line
-	8000 3700 8000 3900
-Wire Wire Line
-	8000 3900 8000 4400
-Connection ~ 8000 3900
-Connection ~ 8000 4400
-Connection ~ 7300 3600
-Wire Wire Line
-	7300 3600 7300 4300
-Wire Wire Line
-	7550 3500 7550 4200
-Connection ~ 7550 4200
+P 9800 3600
+F 0 "J2" H 9850 3917 50  0000 C CNN
+F 1 "Conn_02x03_Odd_Even" H 9850 3826 50  0000 C CNN
+F 2 "Connector_PinHeader_2.54mm:PinHeader_2x03_P2.54mm_Vertical" H 9800 3600 50  0001 C CNN
+F 3 "~" H 9800 3600 50  0001 C CNN
+	1    9800 3600
+	1    0    0    -1
+$EndComp
+Wire Wire Line
+	10100 3500 10350 3500
+Wire Wire Line
+	10350 3500 10350 3900
+NoConn ~ 10100 3600
+NoConn ~ 10100 3700
 Text Label 3450 3950 2    50   ~ 0
 PORTB2
@@
 NoConn ~ 3550 4450
 NoConn ~ 3550 4650
-NoConn ~ 3550 4750
 NoConn ~ 3550 4850
 NoConn ~ 3550 4950
@@
 NoConn ~ 4050 4950
 NoConn ~ 4050 4850
-NoConn ~ 4050 4750
 NoConn ~ 4050 4650
 NoConn ~ 4050 4450
@@
 	5300 3400 5850 3400
 Connection ~ 7300 3300
-Wire Wire Line
-	7300 3300 7300 3600
 $Comp
 L power:GND #PWR0101
@@
 L power:PWR_FLAG #FLG0105
 U 1 1 60D2C30D
-P 2100 2650
-F 0 "#FLG0105" H 2100 2725 50  0001 C CNN
-F 1 "PWR_FLAG" H 2100 2823 50  0000 C CNN
-F 2 "" H 2100 2650 50  0001 C CNN
-F 3 "~" H 2100 2650 50  0001 C CNN
-	1    2100 2650
+P 2050 3800
+F 0 "#FLG0105" H 2050 3875 50  0001 C CNN
+F 1 "PWR_FLAG" H 2050 3973 50  0000 C CNN
+F 2 "" H 2050 3800 50  0001 C CNN
+F 3 "~" H 2050 3800 50  0001 C CNN
+	1    2050 3800
 	1    0    0    -1
 $EndComp
@@
 L power:GND #PWR0103
 U 1 1 60D2C68E
-P 2100 2800
-F 0 "#PWR0103" H 2100 2550 50  0001 C CNN
-F 1 "GND" H 2105 2627 50  0000 C CNN
-F 2 "" H 2100 2800 50  0001 C CNN
-F 3 "" H 2100 2800 50  0001 C CNN
-	1    2100 2800
-	1    0    0    -1
-$EndComp
-Wire Wire Line
-	2100 2650 2100 2800
-Wire Wire Line
-	8000 4600 8000 5150
-Wire Wire Line
-	7550 4200 7550 5500
+P 2050 3950
+F 0 "#PWR0103" H 2050 3700 50  0001 C CNN
+F 1 "GND" H 2055 3777 50  0000 C CNN
+F 2 "" H 2050 3950 50  0001 C CNN
+F 3 "" H 2050 3950 50  0001 C CNN
+	1    2050 3950
+	1    0    0    -1
+$EndComp
+Wire Wire Line
+	2050 3800 2050 3950
+Wire Wire Line
+	9250 4600 9250 5150
 NoConn ~ 2600 5250
 Wire Wire Line
@@
 	2750 5450 2600 5450
 Connection ~ 2750 5250
+Text Label 4150 4750 0    50   ~ 0
+PWM2
+Text Label 3450 4750 2    50   ~ 0
+PWM1
+Wire Wire Line
+	3450 4750 3550 4750
+Wire Wire Line
+	7550 3500 7550 4200
+Wire Wire Line
+	7300 3600 9600 3600
+Wire Wire Line
+	7300 3300 7300 3600
+Connection ~ 7300 3600
+Wire Wire Line
+	7300 3600 7300 4300
+Wire Wire Line
+	7300 4300 9600 4300
+Wire Wire Line
+	7550 3500 9600 3500
+Wire Wire Line
+	7550 4200 9600 4200
+Connection ~ 7550 4200
+Wire Wire Line
+	7550 4200 7550 5500
+Wire Wire Line
+	7200 5150 9250 5150
+$Comp
+L Jumper:Jumper_3_Bridged12 JP1
+U 1 1 60C35BDC
+P 8700 3900
+F 0 "JP1" H 8700 4011 50  0000 C CNN
+F 1 "Jumper_3_Bridged12" H 8700 4102 50  0000 C CNN
+F 2 "Jumper:SolderJumper-3_P1.3mm_Bridged12_RoundedPad1.0x1.5mm" H 8700 3900 50  0001 C CNN
+F 3 "~" H 8700 3900 50  0001 C CNN
+	1    8700 3900
+	-1   0    0    1
+$EndComp
+Wire Wire Line
+	9250 4400 9250 3900
+Wire Wire Line
+	9250 3900 8950 3900
+Connection ~ 9250 4400
+Wire Wire Line
+	8700 3750 8700 3700
+Text Label 7900 3900 2    50   ~ 0
+PWM1
+$Comp
+L Device:R R3
+U 1 1 60C80000
+P 8100 3900
+F 0 "R3" H 8170 3946 50  0000 L CNN
+F 1 "1k" H 8170 3855 50  0000 L CNN
+F 2 "Resistor_SMD:R_0603_1608Metric_Pad1.05x0.95mm_HandSolder" V 8030 3900 50  0001 C CNN
+F 3 "~" H 8100 3900 50  0001 C CNN
+	1    8100 3900
+	0    1    1    0
+$EndComp
+Wire Wire Line
+	7900 3900 7950 3900
+Wire Wire Line
+	8250 3900 8450 3900
+$Comp
+L Jumper:Jumper_3_Bridged12 JP2
+U 1 1 60C88630
+P 8700 4600
+F 0 "JP2" H 8700 4711 50  0000 C CNN
+F 1 "Jumper_3_Bridged12" H 8700 4802 50  0000 C CNN
+F 2 "Jumper:SolderJumper-3_P1.3mm_Bridged12_RoundedPad1.0x1.5mm" H 8700 4600 50  0001 C CNN
+F 3 "~" H 8700 4600 50  0001 C CNN
+	1    8700 4600
+	-1   0    0    1
+$EndComp
+Wire Wire Line
+	9250 4600 8950 4600
+Wire Wire Line
+	8700 4450 8700 4400
+Wire Wire Line
+	8700 4400 9250 4400
+Text Label 7900 4600 2    50   ~ 0
+PWM2
+$Comp
+L Device:R R4
+U 1 1 60C8863A
+P 8100 4600
+F 0 "R4" H 8170 4646 50  0000 L CNN
+F 1 "1k" H 8170 4555 50  0000 L CNN
+F 2 "Resistor_SMD:R_0603_1608Metric_Pad1.05x0.95mm_HandSolder" V 8030 4600 50  0001 C CNN
+F 3 "~" H 8100 4600 50  0001 C CNN
+	1    8100 4600
+	0    1    1    0
+$EndComp
+Wire Wire Line
+	7900 4600 7950 4600
+Wire Wire Line
+	8250 4600 8450 4600
+Wire Wire Line
+	8700 3700 9400 3700
+Wire Wire Line
+	9400 3700 9400 3900
+Wire Wire Line
+	9400 3900 10350 3900
+Connection ~ 9400 3700
+Wire Wire Line
+	9400 3700 9600 3700
+Wire Wire Line
+	9400 4400 9400 4600
+Wire Wire Line
+	9400 4600 10350 4600
+Connection ~ 9400 4400
+Wire Wire Line
+	9400 4400 9600 4400
 $Comp
 L Connector_Generic:Conn_01x04 J4
-U 1 1 60C5F21C
-P 6050 2350
-F 0 "J4" H 6130 2342 50  0000 L CNN
-F 1 "Conn_01x04" H 6130 2251 50  0000 L CNN
-F 2 "Connector_JST:JST_PH_S4B-PH-K_1x04_P2.00mm_Horizontal" H 6050 2350 50  0001 C CNN
-F 3 "~" H 6050 2350 50  0001 C CNN
-	1    6050 2350
-	1    0    0    -1
-$EndComp
-Wire Wire Line
-	5750 2250 5850 2250
-Wire Wire Line
-	5750 2350 5850 2350
+U 1 1 60CA66E1
+P 6050 2200
+F 0 "J4" H 6130 2192 50  0000 L CNN
+F 1 "Conn_01x04" H 6130 2101 50  0000 L CNN
+F 2 "Connector_JST:JST_PH_S4B-PH-K_1x04_P2.00mm_Horizontal" H 6050 2200 50  0001 C CNN
+F 3 "~" H 6050 2200 50  0001 C CNN
+	1    6050 2200
+	1    0    0    -1
+$EndComp
+Wire Wire Line
+	5750 2100 5850 2100
+Wire Wire Line
+	5750 2200 5850 2200
 $Comp
 L power:+5V #PWR01
-U 1 1 60C5F226
-P 5300 2450
-F 0 "#PWR01" H 5300 2300 50  0001 C CNN
-F 1 "+5V" H 5315 2623 50  0000 C CNN
-F 2 "" H 5300 2450 50  0001 C CNN
-F 3 "" H 5300 2450 50  0001 C CNN
-	1    5300 2450
-	1    0    0    -1
-$EndComp
-Wire Wire Line
-	5300 2450 5850 2450
+U 1 1 60CA66EB
+P 5300 2300
+F 0 "#PWR01" H 5300 2150 50  0001 C CNN
+F 1 "+5V" H 5315 2473 50  0000 C CNN
+F 2 "" H 5300 2300 50  0001 C CNN
+F 3 "" H 5300 2300 50  0001 C CNN
+	1    5300 2300
+	1    0    0    -1
+$EndComp
+Wire Wire Line
+	5300 2300 5850 2300
 $Comp
 L power:GND #PWR011
-U 1 1 60C5F22D
-P 5300 2550
-F 0 "#PWR011" H 5300 2300 50  0001 C CNN
-F 1 "GND" H 5305 2377 50  0000 C CNN
-F 2 "" H 5300 2550 50  0001 C CNN
-F 3 "" H 5300 2550 50  0001 C CNN
-	1    5300 2550
-	1    0    0    -1
-$EndComp
-Wire Wire Line
-	5300 2550 5850 2550
-Text Label 5750 2350 2    50   ~ 0
+U 1 1 60CA66F2
+P 5300 2400
+F 0 "#PWR011" H 5300 2150 50  0001 C CNN
+F 1 "GND" H 5305 2227 50  0000 C CNN
+F 2 "" H 5300 2400 50  0001 C CNN
+F 3 "" H 5300 2400 50  0001 C CNN
+	1    5300 2400
+	1    0    0    -1
+$EndComp
+Wire Wire Line
+	5300 2400 5850 2400
+Text Label 5750 2100 2    50   ~ 0
+TXD2
+Text Label 5750 2200 2    50   ~ 0
 RXD2
-Text Label 5750 2250 2    50   ~ 0
-TXD2
+Wire Wire Line
+	4050 4750 4150 4750
 $EndSCHEMATC

Commit message: Add parts
Parts:
- C1: URL (none) -> https://www.sengoku.co.jp/mod/sgk_cart/detail.php?code=46S8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
- J1: URL (none) -> https://www.switch-science.com/catalog/3654/
- J2: URL (none) -> https://akizukidenshi.com/catalog/g/gC-00080/
- J4, R2, R3: URL (none) -> https://www.sengoku.co.jp/mod/sgk_cart/detail.php?code=EEHD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
- J5: URL (none) -> https://akizukidenshi.com/catalog/g/gC-12802/
Changed lines of the file:
@@
 F 2 "m5-pantilt:NL27WZ125USG" H 5500 5650 50  0001 C CNN
 F 3 "" H 5500 5650 50  0001 C CNN
+F 4 "" H 5750 5250 50  0001 C CNN "URL"
 	1    5750 5250
 	1    0    0    -1
@@
 F 2 "Connector_PinHeader_2.54mm:PinHeader_2x15_P2.54mm_Vertical_SMD" H 3750 4550 50  0001 C CNN
 F 3 "~" H 3750 4550 50  0001 C CNN
+F 4 "https://www.switch-science.com/catalog/3654/" H 3750 4550 50  0001 C CNN "URL"
 	1    3750 4550
 	1    0    0    -1
@@
 F 2 "Resistor_SMD:R_0603_1608Metric_Pad1.05x0.95mm_HandSolder" V 6980 5150 50  0001 C CNN
 F 3 "~" H 7050 5150 50  0001 C CNN
+F 4 "https://www.sengoku.co.jp/mod/sgk_cart/detail.php?code=EEHD-57FV" V 7050 5150 50  0001 C CNN "URL"
 	1    7050 5150
 	0    1    1    0
@@
 F 2 "Connector_PinHeader_2.54mm:PinHeader_2x03_P2.54mm_Vertical" H 9800 3600 50  0001 C CNN
 F 3 "~" H 9800 3600 50  0001 C CNN
+F 4 "https://akizukidenshi.com/catalog/g/gC-00080/" H 9800 3600 50  0001 C CNN "URL"
 	1    9800 3600
 	1    0    0    -1
@@
 F 2 "Connector_JST:JST_PH_B2B-PH-K_1x02_P2.00mm_Vertical" H 2000 5350 50  0001 C CNN
 F 3 "~" H 2000 5350 50  0001 C CNN
+F 4 "https://akizukidenshi.com/catalog/g/gC-12802/" H 2000 5350 50  0001 C CNN "URL"
 	1    2000 5350
 	-1   0    0    -1
@@
 F 2 "Capacitor_THT:C_Radial_D6.3mm_H11.0mm_P2.50mm" H 7188 3150 50  0001 C CNN
 F 3 "~" H 7150 3300 50  0001 C CNN
+F 4 "https://www.sengoku.co.jp/mod/sgk_cart/detail.php?code=46S8-5GL7" V 7150 3300 50  0001 C CNN "URL"
 	1    7150 3300
 	0    -1   -1   0
@@
 F 2 "Resistor_SMD:R_0603_1608Metric_Pad1.05x0.95mm_HandSolder" V 8030 3900 50  0001 C CNN
 F 3 "~" H 8100 3900 50  0001 C CNN
+F 4 "https://www.sengoku.co.jp/mod/sgk_cart/detail.php?code=EEHD-57GK" H 8100 3900 50  0001 C CNN "URL"
 	1    8100 3900
 	0    1    1    0
@@
 F 2 "Connector_JST:JST_PH_S4B-PH-K_1x04_P2.00mm_Horizontal" H 6050 2200 50  0001 C CNN
 F 3 "~" H 6050 2200 50  0001 C CNN
+F 4 "https://www.sengoku.co.jp/mod/sgk_cart/detail.php?code=EEHD-55FC" H 6050 2200 50  0001 C CNN "URL"
 	1    6050 2200
 	1    0    0    -1
