File: schematics/m5-pantilt/m5-pantilt.kicad_pcb (KiCad board)
At the start: 2 copper layers, 50 x 50 mm, 37 parts, among them J1 Conn_02x15_Odd_Even, J2 Conn_02x03_Odd_Even, J3 Conn_02x03_Odd_Even, J4 Conn_01x04, J5 BAT, J6 Conn_01x04, J7 5V_POWER, Q1 IRLML6402, SW1 SW_SPDT, U1 TC7WH241FK

Commit message: fix schematics
Parts:
- removed JP10, JP9: Jumper_2_Open, Jumper:SolderJumper-2_P1.3mm_Open_Pad1.0x1.5mm
- removed R7, R8: 0, Resistor_SMD:R_0603_1608Metric_Pad1.05x0.95mm_HandSolder
- moved R13 52.9 mm to (123.3, 86.9)
- moved R9 51.8 mm to (115.8, 81.1), turned to 180 degrees
- moved R6 51.2 mm to (115.7, 72.8)
- moved R15 49.9 mm to (123.4, 72.8)
- moved R10 49.3 mm to (115.8, 85.2), turned to 180 degrees
- moved R12 49.0 mm to (115.8, 86.8), turned to 180 degrees
- moved R16 45.5 mm to (123.4, 71.0), turned to 180 degrees
- moved R11 45.2 mm to (115.8, 82.7), turned to 180 degrees
- moved R14 19.5 mm to (123.3, 85.2), turned to 180 degrees
Connections:
- R3 pad 1: Net-(R3-Pad1) -> Net-(J2-Pad2)
- R4 pad 1: Net-(R4-Pad1) -> Net-(J3-Pad2)
Routing:
- net Net-(J3-Pad2): track 6.47 -> 31.2 mm, vias 0 -> 1
- net Net-(J2-Pad2): track 18.9 -> 29.0 mm, vias 0 -> 1
- net Net-(R14-Pad1): track 0.00 -> 9.34 mm, vias 0 -> 2
- net Net-(R3-Pad1): track 9.14 -> 0.00 mm, vias 1 -> 0
- net Net-(R4-Pad1): track 8.55 -> 0.00 mm, vias 1 -> 0
- net Net-(R15-Pad1): track 0.00 -> 7.92 mm
- net Net-(JP10-Pad2): track 7.92 -> 0.00 mm
- net /PWM2_C2: track 11.2 -> 17.8 mm, vias 0 -> 1
- net /PWM2_C1: track 12.7 -> 17.6 mm, vias 0 -> 1
- net /PWM1: track 10.8 -> 15.5 mm, vias 1 -> 0
- net +3V3: track 25.1 -> 28.4 mm
- net /TXD2: track 30.8 -> 32.9 mm, vias 2 -> 3
- net /PWM1_C2: track 5.87 -> 7.20 mm, vias 0 -> 1
- net /PWM1_C1: track 5.81 -> 6.57 mm, vias 0 -> 1
- net /PWM2: track 15.0 -> 14.6 mm, vias 1 -> 0
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Other:
- board text added: "Core1PWM"
- board text added: "Core2PWM"
- board text added: "U1's 7th pin TC7WH251(pull-up): R16 TC7WH241(pull-down): R15"
- board text removed: "Anode"
- board text removed: "Cathode"
- board text removed: "Core1"
- board text removed: "Core2"
- board text removed: "PWM"
- board text removed: "U1's 7th pin pull-up: JP10 pull-down: JP9"

Commit message: fix schematics
Routing:
- net /PWM2_C1: track 17.6 -> 12.3 mm
- net /PWM2_C2: track 17.8 -> 12.9 mm
- net GND: vias 103 -> 105
Other:
- board text added: "U1's 7th pin Inverted : R16(pull-up) Non inverted: R15(pull-down)"
- board text removed: "U1's 7th pin TC7WH251(pull-up): R16 TC7WH241(pull-down): R15"
