File: schematics/m5-pantilt/m5-pantilt.kicad_pcb (KiCad board)
At the start: 2 copper layers, 50 x 50 mm, 38 parts, among them J1 Conn_02x15_Odd_Even, J2 Conn_02x15_Odd_Even, J3 Conn_01x03, J4 Conn_01x04, J5 BAT, J6 Conn_01x04, J7 5V_POWER, J8 Conn_01x03, Q1 IRLML6402, Q2 2SA1015, SW1 SW_SPDT, U1 MAX3485

Commit message: Update board
Parts:
- Q2: value 2SA1015 -> BC857; footprint m5-pantilt:2SA1015_SOT-23 -> Package_TO_SOT_SMD:SOT-23
- R2: value 7.5k -> 5k
- moved R1 7.51 mm to (115.5, 71.6), turned to -90 degrees
- moved R2 6.12 mm to (117.0, 71.6), turned to 90 degrees
- moved R7 5.38 mm to (116.2, 65.8)
- moved J5 0.32 mm to (142.3, 91.2)
- turned Q2 to 0 degrees
Connections:
- Q2 pad 1: Net-(Q2-Pad1) -> Net-(R2-Pad2)
- Q2 pad 3: Net-(Q2-Pad3) -> Net-(R7-Pad1)
- R2 pad 2: Net-(Q2-Pad3) -> Net-(R2-Pad2)
- R7 pad 1: Net-(Q2-Pad1) -> Net-(R7-Pad1)
- U1 pad 2: Net-(Q2-Pad1) -> Net-(R7-Pad1)
- U1 pad 3: Net-(Q2-Pad1) -> Net-(R7-Pad1)
Routing:
- net Net-(Q2-Pad1): track 7.47 -> 0.00 mm
- net Net-(R7-Pad1): track 0.00 -> 6.88 mm
- net Net-(R2-Pad2): track 0.00 -> 4.31 mm
- net /TXD2: track 43.0 -> 39.4 mm, vias 3 -> 1
- net Net-(Q2-Pad3): track 2.00 -> 0.00 mm
- net /RXD2: track 43.6 -> 41.6 mm
- net +3V3: track 41.1 -> 39.7 mm
- net Net-(J3-Pad3): track 38.6 -> 37.6 mm
- net GND: vias 62 -> 69

Commit message: 5k->5.1k
Parts:
- R2: value 5k -> 5.1k
Changed lines of the file:
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@@
       (effects (font (size 1 1) (thickness 0.15)))
     )
-    (fp_text value "5k" (at 0 1.43 90) (layer "F.Fab")
+    (fp_text value "5.1k" (at 0 1.43 90) (layer "F.Fab")
       (effects (font (size 1 1) (thickness 0.15)))
     )

Commit message: Improve power function of the board
Parts:
- removed J4: Conn_01x04, Connector_JST:JST_PH_S4B-PH-K_1x04_P2.00mm_Horizontal
- added D2: PMEG3030EP, Diode_SMD:D_SOD-128, F.Cu at (136.8, 63.4)
- D1: value D -> SS54
- SW1: moved to F.Cu
- moved D1 39.9 mm to (124.5, 53.2), turned to 180 degrees
- moved J7 37.8 mm to (118.0, 54.5), turned to 180 degrees
- moved SW1 4.05 mm to (145.8, 63.1), turned to 90 degrees
Connections:
- C1 pad 2: +5V -> Net-(D2-K)
- C2 pad 2: +5V -> Net-(D2-K)
- C3 pad 1: +5V -> Net-(D2-K)
- C4 pad 2: +5V -> Net-(D2-K)
- J3 pad 2: +5V -> Net-(D2-K)
- J8 pad 2: +5V -> Net-(D2-K)
- SW1 pad 1: GND -> unconnected-(SW1-A-Pad1)
- SW1 pad 3: unconnected-(SW1-C-Pad3) -> GND
Routing:
- net Net-(D2-K): track 0.00 -> 37.4 mm
- net +5V: track 102.8 -> 74.0 mm, vias 1 -> 2
- net /TXD2: track 39.4 -> 17.6 mm
- net /RXD2: track 41.6 -> 23.4 mm, vias 4 -> 2
- net /BAT: track 29.7 -> 26.0 mm
- net Net-(J5-Pin_1): track 11.2 -> 12.9 mm
- net Net-(J8-Pin_3): track 47.7 -> 49.2 mm
- net Net-(J3-Pin_3): track 37.6 -> 38.4 mm
- net GND: vias 69 -> 79
Other:
- board text added: "m5-pantilt board v1.0.0rc @meganetaaan"
- board text removed: "RX"
- board text removed: "TX"
- board text removed: "UART"
- board text removed: "m5-pantilt board v0.2.1 @meganetaaan"
