File: schematics/m5-pantilt/m5-pantilt.kicad_sch (KiCad schematic)
At the start: 33 parts, among them J1 Conn_02x15_Odd_Even, J2 Conn_02x15_Odd_Even, J3 Conn_01x03, J4 Conn_01x04, J5 BAT, J6 Conn_01x04, J7 5V_POWER, J8 Conn_01x03, Q1 IRLML6402, Q2 BC857, SW1 SW_SPDT, U1 MAX3485

Commit message: Add LCSC part number
Parts:
- C1, C2, C3, C4: LCSC (none) -> C15008
- C5: LCSC (none) -> C14663
- D1: LCSC (none) -> C2931790
- J6: URL (none) -> https://www.sengoku.co.jp/mod/sgk_cart/detail.php?code=EEHD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
- J7: LCSC (none) -> C20079
- Q1: LCSC (none) -> C2886430
- Q2: LCSC (none) -> C2139
- R1: LCSC (none) -> C25804
- R10, R11, R12, R13, R14, R9: LCSC (none) -> C21189
- R15, R8: LCSC (none) -> C4190
- R2: LCSC (none) -> C23186
- R3: LCSC (none) -> C21190
- R4: LCSC (none) -> C21190; URL (none) -> https://www.sengoku.co.jp/mod/sgk_cart/detail.php?code=EEHD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
- R5: LCSC (none) -> C25819
- R6: LCSC (none) -> C22975
- R7: LCSC (none) -> C4184
- U1: LCSC (none) -> C668204
Changed lines of the file:
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@@
+      (effects (font (size 1.27 1.27)) hide)
+    )
+    (property "LCSC" "C21190" (at 205.74 99.06 0)
       (effects (font (size 1.27 1.27)) hide)
     )
@@
       (effects (font (size 1.27 1.27)) hide)
     )
+    (property "LCSC" "C21190" (at 205.74 125.73 0)
+      (effects (font (size 1.27 1.27)) hide)
+    )
+    (property "URL" "https://www.sengoku.co.jp/mod/sgk_cart/detail.php?code=EEHD-57GK" (at 205.74 125.73 0)
+      (effects (font (size 1.27 1.27)) hide)
+    )
     (pin "1")
     (pin "2")
@@
     )
     (property "Datasheet" "~" (at 149.86 81.28 0)
+      (effects (font (size 1.27 1.27)) hide)
+    )
+    (property "URL" "https://www.sengoku.co.jp/mod/sgk_cart/detail.php?code=EEHD-55FC" (at 149.86 81.28 0)
       (effects (font (size 1.27 1.27)) hide)
     )
@@
       (effects (font (size 1.27 1.27)) hide)
     )
+    (property "LCSC" "C15008" (at 219.71 87.63 0)
+      (effects (font (size 1.27 1.27)) hide)
+    )
     (pin "1")
     (pin "2")
@@
       (effects (font (size 1.27 1.27)) hide)
     )
+    (property "LCSC" "C20079" (at 20.32 109.22 0)
+      (effects (font (size 1.27 1.27)) hide)
+    )
     (pin "1")
     (pin "2")
@@
     )
     (property "URL" "https://akizukidenshi.com/catalog/g/gP-15633/" (at 219.71 113.03 90)
+      (effects (font (size 1.27 1.27)) hide)
+    )
+    (property "LCSC" "C15008" (at 219.71 113.03 0)
       (effects (font (size 1.27 1.27)) hide)
     )
@@
       (effects (font (size 1.27 1.27)) hide)
     )
+    (property "LCSC" "C2886430" (at 44.45 135.89 90)
+      (effects (font (size 1.27 1.27)) hide)
+    )
     (pin "1")
     (pin "2")
@@
       (effects (font (size 1.27 1.27)) hide)
     )
+    (property "LCSC" "C25819" (at 34.29 143.51 0)
+      (effects (font (size 1.27 1.27)) hide)
+    )
     (pin "1")
     (pin "2")
@@
       (effects (font (size 1.27 1.27)) hide)
     )
+    (property "LCSC" "C15008" (at 208.28 87.63 0)
+      (effects (font (size 1.27 1.27)) hide)
+    )
     (pin "1")
     (pin "2")
@@
       (effects (font (size 1.27 1.27)) hide)
     )
+    (property "LCSC" "C15008" (at 208.28 113.03 0)
+      (effects (font (size 1.27 1.27)) hide)
+    )
     (pin "1")
     (pin "2")
@@
       (effects (font (size 1.27 1.27)) hide)
     )
+    (property "LCSC" "C21189" (at 220.98 38.1 90)
+      (effects (font (size 1.27 1.27)) hide)
+    )
     (pin "1")
     (pin "2")
@@
       (effects (font (size 1.27 1.27)) hide)
     )
+    (property "LCSC" "C21189" (at 220.98 46.99 90)
+      (effects (font (size 1.27 1.27)) hide)
+    )
     (pin "1")
     (pin "2")
@@
       (effects (font (size 1.27 1.27)) hide)
     )
+    (property "LCSC" "C21189" (at 220.98 55.88 90)
+      (effects (font (size 1.27 1.27)) hide)
+    )
     (pin "1")
     (pin "2")
@@
       (effects (font (size 1.27 1.27)) hide)
     )
+    (property "LCSC" "C21189" (at 220.98 64.77 90)
+      (effects (font (size 1.27 1.27)) hide)
+    )
     (pin "1")
     (pin "2")
@@
       (effects (font (size 1.27 1.27)) hide)
     )
+    (property "LCSC" "C21189" (at 229.87 99.06 90)
+      (effects (font (size 1.27 1.27)) hide)
+    )
     (pin "1")
     (pin "2")
@@
       (effects (font (size 1.27 1.27)) hide)
     )
+    (property "LCSC" "C21189" (at 229.87 125.73 90)
+      (effects (font (size 1.27 1.27)) hide)
+    )
     (pin "1")
     (pin "2")
@@
     )
     (property "Datasheet" "https://datasheets.maximintegrated.com/en/ds/MAX3483-MAX3491.pdf" (at 123.19 134.62 0)
+      (effects (font (size 1.27 1.27)) hide)
+    )
+    (property "LCSC" "C668204" (at 123.19 135.89 0)
       (effects (font (size 1.27 1.27)) hide)
     )
@@
       (effects (font (size 1.27 1.27)) hide)
     )
+    (property "LCSC" "C14663" (at 146.05 127 0)
+      (effects (font (size 1.27 1.27)) hide)
+    )
     (pin "1")
     (pin "2")
@@
       (effects (font (size 1.27 1.27)) hide)
     )
+    (property "LCSC" "C4190" (at 157.48 128.27 0)
+      (effects (font (size 1.27 1.27)) hide)
+    )
     (pin "1")
     (pin "2")
@@
       (effects (font (size 1.27 1.27)) hide)
     )
+    (property "LCSC" "C4190" (at 157.48 142.24 0)
+      (effects (font (size 1.27 1.27)) hide)
+    )
     (pin "1")
     (pin "2")
@@
       (effects (font (size 1.27 1.27)) hide)
     )
+    (property "LCSC" "C4184" (at 95.25 146.05 0)
+      (effects (font (size 1.27 1.27)) hide)
+    )
     (pin "1")
     (pin "2")
@@
     )
     (property "Datasheet" "~" (at 43.18 109.22 0)
+      (effects (font (size 1.27 1.27)) hide)
+    )
+    (property "LCSC" "C2931790" (at 43.18 109.22 0)
       (effects (font (size 1.27 1.27)) hide)
     )
@@
       (effects (font (size 1.27 1.27)) hide)
     )
+    (property "LCSC" "C25804" (at 71.12 120.65 0)
+      (effects (font (size 1.27 1.27)) hide)
+    )
     (pin "1")
     (pin "2")
@@
       (effects (font (size 1.27 1.27)) hide)
     )
+    (property "LCSC" "C23186" (at 81.28 129.54 90)
+      (effects (font (size 1.27 1.27)) hide)
+    )
     (pin "1")
     (pin "2")
@@
       (effects (font (size 1.27 1.27)) hide)
     )
+    (property "LCSC" "C22975" (at 137.16 127 0)
+      (effects (font (size 1.27 1.27)) hide)
+    )
     (pin "1")
     (pin "2")
@@
       (effects (font (size 1.27 1.27)) (justify left) hide)
     )
-    (pin "1")
+    (property "LCSC" "C2139" (at 92.71 129.54 0)
+      (effects (font (size 1.27 1.27)) hide)
+    )
+    (pin "1")

Commit message: Improve power function of the board
Parts:
- removed J4: Conn_01x04, Connector_JST:JST_PH_S4B-PH-K_1x04_P2.00mm_Horizontal, symbol Connector_Generic:Conn_01x04
- added D2: PMEG3030EP, Diode_SMD:D_SOD-128, symbol Device:D_Schottky
- D1: value D -> SS54
Connections:
- net +5V: now also D2.2 (A); no longer C1.2, C2.2, C3.1, C4.2, J3.2 (Pin_2), J8.2 (Pin_2)
- net GND: now also SW1.3 (C); no longer SW1.1 (A)
- new net: C1.2, C2.2, C3.1, C4.2, D2.1 (K), J3.2 (Pin_2), J8.2 (Pin_2)
Other:
- note added: "3A 360mV"
- note added: "forward voltage > 0.6V"
- note removed: "UART"
- moved on the sheet: SW1
Changed lines of the file:
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@@
   (junction (at 123.19 151.13) (diameter 0) (color 0 0 0 0)
   )
+  (junction (at 185.42 83.82) (diameter 0) (color 0 0 0 0)
+  )
   (junction (at 223.52 125.73) (diameter 0) (color 0 0 0 0)
   )
@@
   (junction (at 69.85 101.6) (diameter 0) (color 0 0 0 0)
   )
-  (junction (at 185.42 83.82) (diameter 0) (color 0 0 0 0)
-  )
   (junction (at 55.88 30.48) (diameter 0) (color 0 0 0 0)
   )
@@
     (stroke (width 0) (type default))
   )
+  (wire (pts (xy 185.42 78.74) (xy 185.42 83.82))
+    (stroke (width 0) (type default))
+  )
   (wire (pts (xy 27.94 78.74) (xy 27.94 82.55))
     (stroke (width 0) (type default))
@@
     (stroke (width 0) (type default))
   )
-  (wire (pts (xy 154.94 55.88) (xy 158.75 55.88))
-    (stroke (width 0) (type default))
-  )
   (wire (pts (xy 97.79 76.2) (xy 100.33 76.2))
     (stroke (width 0) (type default))
@@
     (stroke (width 0) (type default))
   )
-  (wire (pts (xy 154.94 60.96) (xy 167.64 60.96))
-    (stroke (width 0) (type default))
-  )
   (wire (pts (xy 232.41 64.77) (xy 232.41 55.88))
     (stroke (width 0) (type default))
@@
     (stroke (width 0) (type default))
   )
-  (wire (pts (xy 185.42 72.39) (xy 185.42 83.82))
-    (stroke (width 0) (type default))
-  )
   (wire (pts (xy 191.77 81.28) (xy 243.84 81.28))
     (stroke (width 0) (type default))
@@
     (stroke (width 0) (type default))
   )
+  (wire (pts (xy 185.42 68.58) (xy 185.42 71.12))
+    (stroke (width 0) (type default))
+  )
   (wire (pts (xy 62.23 129.54) (xy 71.12 129.54))
     (stroke (width 0) (type default))
@@
     (stroke (width 0) (type default))
   )
-  (wire (pts (xy 154.94 58.42) (xy 167.64 58.42))
-    (stroke (width 0) (type default))
-  )
   (wire (pts (xy 154.94 83.82) (xy 167.64 83.82))
     (stroke (width 0) (type default))
@@
     (stroke (width 0) (type default))
   )
-  (wire (pts (xy 154.94 53.34) (xy 158.75 53.34))
-    (stroke (width 0) (type default))
-  )
   (wire (pts (xy 233.68 99.06) (xy 234.95 99.06))
     (stroke (width 0) (type default))
@@
     )
   )
-  (text "UART" (at 147.32 49.53 0)
-    (effects (font (size 1.27 1.27)) (justify left bottom))
-  )
   (text "M-BUS" (at 146.05 72.39 0)
     (effects (font (size 1.27 1.27)) (justify left bottom))
@@
     (effects (font (size 1.27 1.27)) (justify left bottom))
   )
+  (text "forward voltage > 0.6V" (at 35.56 114.3 0)
+    (effects (font (size 1.27 1.27)) (justify left bottom))
+  )
+  (text "3A 360mV" (at 187.96 80.01 0)
+    (effects (font (size 1.27 1.27)) (justify left bottom))
+  )
   (text "Short R10, R10 for Core2 and CoreS3\nShort R9, R11 for others"
     (at 204.47 30.48 0)
@@
     (effects (font (size 1.27 1.27)) (justify left bottom))
   )
-  (label "TXD2" (at 158.75 55.88 0) (fields_autoplaced)
-    (effects (font (size 1.27 1.27)) (justify left bottom))
-  )
   (label "PORTB1" (at 27.94 38.1 180) (fields_autoplaced)
     (effects (font (size 1.27 1.27)) (justify right bottom))
@@
     (effects (font (size 1.27 1.27)) (justify right bottom))
   )
-  (label "RXD2" (at 158.75 53.34 0) (fields_autoplaced)
-    (effects (font (size 1.27 1.27)) (justify left bottom))
-  )
   (label "BAT" (at 57.15 138.43 0) (fields_autoplaced)
     (effects (font (size 1.27 1.27)) (justify left bottom))
@@
     (effects (font (size 1.27 1.27)) (justify right bottom))
   )
-  (label "forward voltage > 0.6V" (at 33.02 114.3 0) (fields_autoplaced)
-    (effects (font (size 1.27 1.27)) (justify left bottom))
-  )
   (label "PIN23" (at 27.94 55.88 180) (fields_autoplaced)
     (effects (font (size 1.27 1.27)) (justify right bottom))
@@
     )
   )
-  (symbol (lib_id "power:+5V") (at 185.42 72.39 0) (unit 1)
+  (symbol (lib_id "power:+5V") (at 185.42 68.58 0) (unit 1)
     (in_bom yes) (on_board yes) (dnp no)
-    (property "Reference" "#PWR07" (at 185.42 76.2 0)
+    (property "Reference" "#PWR07" (at 185.42 72.39 0)
       (effects (font (size 1.27 1.27)) hide)
     )
-    (property "Value" "+5V" (at 185.801 67.9958 0)
+    (property "Value" "+5V" (at 185.801 64.1858 0)
       (effects (font (size 1.27 1.27)))
     )
-    (property "Footprint" "" (at 185.42 72.39 0)
+    (property "Footprint" "" (at 185.42 68.58 0)
       (effects (font (size 1.27 1.27)) hide)
     )
-    (property "Datasheet" "" (at 185.42 72.39 0)
+    (property "Datasheet" "" (at 185.42 68.58 0)
       (effects (font (size 1.27 1.27)) hide)
     )
@@
     )
   )
-  (symbol (lib_id "Connector_Generic:Conn_01x04") (at 149.86 58.42 180) (unit 1)
-    (in_bom yes) (on_board yes) (dnp no)
-    (property "Reference" "J4" (at 147.828 58.2168 0)
-      (effects (font (size 1.27 1.27)) (justify left))
-    )
-    (property "Value" "Conn_01x04" (at 147.828 55.9054 0)
-      (effects (font (size 1.27 1.27)) (justify left))
-    )
-    (property "Footprint" "Connector_JST:JST_PH_S4B-PH-K_1x04_P2.00mm_Horizontal" (at 149.86 58.42 0)
-      (effects (font (size 1.27 1.27)) hide)
-    )
-    (property "Datasheet" "~" (at 149.86 58.42 0)
-      (effects (font (size 1.27 1.27)) hide)
-    )
-    (property "URL" "https://www.sengoku.co.jp/mod/sgk_cart/detail.php?code=EEHD-55FC" (at 149.86 58.42 0)
-      (effects (font (size 1.27 1.27)) hide)
-    )
-    (pin "1")
-    (pin "2")
-    (pin "3")
-    (pin "4")
-    (instances
-      (project "m5-pantilt"
-        (path "/a27eb049-c992-4f11-a026-1e6a8d9d0160"
-          (reference "J4") (unit 1)
-        )
-      )
-    )
-  )
-  (symbol (lib_id "power:+5V") (at 167.64 58.42 0) (unit 1)
-    (in_bom yes) (on_board yes) (dnp no)
-    (property "Reference" "#PWR01" (at 167.64 62.23 0)
-      (effects (font (size 1.27 1.27)) hide)
-    )
-    (property "Value" "+5V" (at 168.021 54.0258 0)
-      (effects (font (size 1.27 1.27)))
-    )
-    (property "Footprint" "" (at 167.64 58.42 0)
-      (effects (font (size 1.27 1.27)) hide)
-    )
-    (property "Datasheet" "" (at 167.64 58.42 0)
-      (effects (font (size 1.27 1.27)) hide)
-    )
-    (pin "1")
-    (instances
-      (project "m5-pantilt"
-        (path "/a27eb049-c992-4f11-a026-1e6a8d9d0160"
-          (reference "#PWR01") (unit 1)
-        )
-      )
-    )
-  )
-  (symbol (lib_id "power:GND") (at 167.64 60.96 0) (unit 1)
-    (in_bom yes) (on_board yes) (dnp no)
-    (property "Reference" "#PWR011" (at 167.64 67.31 0)
-      (effects (font (size 1.27 1.27)) hide)
-    )
-    (property "Value" "GND" (at 167.767 65.3542 0)
-      (effects (font (size 1.27 1.27)))
-    )
-    (property "Footprint" "" (at 167.64 60.96 0)
-      (effects (font (size 1.27 1.27)) hide)
-    )
-    (property "Datasheet" "" (at 167.64 60.96 0)
-      (effects (font (size 1.27 1.27)) hide)
-    )
-    (pin "1")
-    (instances
-      (project "m5-pantilt"
-        (path "/a27eb049-c992-4f11-a026-1e6a8d9d0160"
-          (reference "#PWR011") (unit 1)
-        )
-      )
-    )
-  )
   (symbol (lib_id "Device:C") (at 219.71 87.63 180) (unit 1)
     (in_bom yes) (on_board yes) (dnp no)
@@
     )
   )
-  (symbol (lib_id "Switch:SW_SPDT") (at 34.29 156.21 270) (unit 1)
+  (symbol (lib_id "Switch:SW_SPDT") (at 34.29 156.21 90) (mirror x) (unit 1)
     (in_bom yes) (on_board yes) (dnp no)
     (property "Reference" "SW1" (at 41.91 158.75 90)
       (effects (font (size 1.27 1.27)))
     )
-    (property "Value" "SW_SPDT" (at 40.64 156.21 90)
+    (property "Value" "SW_SPDT" (at 41.91 156.21 90)
       (effects (font (size 1.27 1.27)))
     )
@@
       (effects (font (size 1.27 1.27)))
     )
-    (property "Value" "D" (at 43.18 106.045 0)
+    (property "Value" "SS54" (at 43.18 106.045 0)
       (effects (font (size 1.27 1.27)))
     )
@@
         )
       )
+    )
+  )
+  (symbol (lib_id "Device:D_Schottky") (at 185.42 74.93 90) (unit 1)
+    (in_bom yes) (on_board yes) (dnp no) (fields_autoplaced)
+    (property "Reference" "D2" (at 187.96 73.9775 90)
+      (effects (font (size 1.27 1.27)) (justify right))
+    )
+    (property "Value" "PMEG3030EP" (at 187.96 76.5175 90)
+      (effects (font (size 1.27 1.27)) (justify right))
+    )
+    (property "Footprint" "Diode_SMD:D_SOD-128" (at 185.42 74.93 0)
+      (effects (font (size 1.27 1.27)) hide)
+    )
+    (property "Datasheet" "~" (at 185.42 74.93 0)
+      (effects (font (size 1.27 1.27)) hide)
+    )
+    (property "LCSC" "C255587" (at 185.42 74.93 90)
+      (effects (font (size 1.27 1.27)) hide)
+    )
+    (pin "1")
+    (pin "2")
+    (instances
+      (project "m5-pantilt"
+        (path "/a27eb049-c992-4f11-a026-1e6a8d9d0160"
+          (reference "D2") (unit 1)
+        )
+      )

Commit message: WIP: fix board
Parts:
- removed D1: SS54, Diode_SMD:D_SMA, symbol Device:D
- removed J7: 5V_POWER, Connector_JST:JST_XH_B2B-XH-A_1x02_P2.50mm_Vertical, symbol Connector_Generic:Conn_01x02
- added J4: PortC, Connector_JST:JST_PH_S4B-PH-K_1x04_P2.00mm_Horizontal, symbol Connector_Generic:Conn_01x04
- added R16: 5.1k, Resistor_SMD:R_0603_1608Metric_Pad0.98x0.95mm_HandSolder, symbol Device:R
- added R17, R18: 0, Resistor_SMD:R_0603_1608Metric_Pad0.98x0.95mm_HandSolder, symbol Device:R
- J6: value Conn_01x04 -> PortB
Connections:
- net +5V: now also J4.2 (Pin_2), R16.2
- net GND: now also J4.1 (Pin_1), R16.1
- net RXD2: now also J4.4 (Pin_4), R18.2; no longer U1.1 (RO)
- net TXD2: now also J4.3 (Pin_3), R17.2; no longer R1.2, R2.1, U1.4 (DI)
- net PWM1 renamed SERVO1
- net SERVO1: now also R1.2, R2.1, U1.4 (DI), R17.1
- net PWM2 renamed SERVO2
- net SERVO2: now also U1.1 (RO), R18.1
Other:
- note removed: "forward voltage > 0.6V"
- moved on the sheet: R10, R9
